File: hardware/UPP_simple/adc.kicad_sch (KiCad schematic)
At the start: 3 parts, among them IC1 ADS114S08BIPBSR

Commit message: Add files via upload
Parts:
- C1, C2: footprint (none) -> Capacitor_SMD:C_0603_1608Metric_Pad1.08x0.95mm_HandSolder
Connections:
- net ADC.CLK renamed ADC_SPI.CLK
- net ADC.CS renamed ADC_SPI.CS
- net ADC.MISO renamed ADC_SPI.MISO
- net ADC.MOSI renamed ADC_SPI.MOSI
- no-connect marks 0 -> 5
Changed lines of the file:
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@@
 		(color 0 0 0 0)
+	)
+	(no_connect
+		(at 143.51 60.96)
+	)
+	(no_connect
+		(at 153.67 124.46)
+	)
+	(no_connect
+		(at 125.73 83.82)
+	)
+	(no_connect
+		(at 156.21 124.46)
+	)
+	(no_connect
+		(at 146.05 60.96)
 	)
 	(bus_entry
@@
 	)
 	(bus_entry
-		(at 138.43 134.62)
+		(at 138.43 138.43)
 		(size 2.54 2.54)
 		(stroke
@@
 	)
 	(bus_entry
-		(at 115.57 101.6)
-		(size -2.54 2.54)
-		(stroke
-			(width 0)
-			(type default)
-		)
-	)
-	(bus_entry
-		(at 140.97 134.62)
+		(at 140.97 138.43)
 		(size 2.54 2.54)
 		(stroke
@@
 	)
 	(bus_entry
-		(at 180.34 99.06)
-		(size 2.54 -2.54)
-		(stroke
-			(width 0)
-			(type default)
-		)
-	)
-	(bus_entry
 		(at 120.65 96.52)
 		(size -2.54 -2.54)
@@
 	)
 	(bus_entry
-		(at 148.59 134.62)
+		(at 143.51 138.43)
 		(size 2.54 2.54)
 		(stroke
@@
 	)
 	(bus_entry
-		(at 143.51 134.62)
-		(size 2.54 2.54)
-		(stroke
-			(width 0)
-			(type default)
-		)
-	)
-	(bus_entry
-		(at 146.05 134.62)
+		(at 146.05 138.43)
 		(size 2.54 2.54)
 		(stroke
@@
 	(wire
 		(pts
-			(xy 140.97 124.46) (xy 140.97 134.62)
+			(xy 140.97 124.46) (xy 140.97 138.43)
 		)
 		(stroke
@@
 		)
 	)
-	(bus
-		(pts
-			(xy 182.88 137.16) (xy 151.13 137.16)
-		)
-		(stroke
-			(width 0)
-			(type default)
-		)
-	)
-	(wire
-		(pts
-			(xy 171.45 99.06) (xy 180.34 99.06)
-		)
-		(stroke
-			(width 0)
-			(type default)
-		)
-	)
-	(bus
-		(pts
-			(xy 140.97 137.16) (xy 113.03 137.16)
+	(wire
+		(pts
+			(xy 171.45 99.06) (xy 185.42 99.06)
 		)
 		(stroke
@@
 	(bus
 		(pts
-			(xy 148.59 137.16) (xy 146.05 137.16)
+			(xy 148.59 140.97) (xy 146.05 140.97)
 		)
 		(stroke
@@
 	(wire
 		(pts
-			(xy 146.05 124.46) (xy 146.05 134.62)
-		)
-		(stroke
-			(width 0)
-			(type default)
-		)
-	)
-	(wire
-		(pts
-			(xy 143.51 124.46) (xy 143.51 134.62)
+			(xy 146.05 124.46) (xy 146.05 138.43)
+		)
+		(stroke
+			(width 0)
+			(type default)
+		)
+	)
+	(wire
+		(pts
+			(xy 143.51 124.46) (xy 143.51 138.43)
 		)
 		(stroke
@@
 	(bus
 		(pts
+			(xy 137.16 143.51) (xy 140.97 143.51)
+		)
+		(stroke
+			(width 0)
+			(type default)
+		)
+	)
+	(bus
+		(pts
 			(xy 179.07 83.82) (xy 179.07 86.36)
 		)
@@
 		)
 	)
-	(wire
-		(pts
-			(xy 138.43 124.46) (xy 138.43 134.62)
-		)
-		(stroke
-			(width 0)
-			(type default)
-		)
-	)
 	(bus
 		(pts
@@
 		)
 	)
-	(bus
-		(pts
-			(xy 113.03 104.14) (xy 113.03 137.16)
-		)
-		(stroke
-			(width 0)
-			(type default)
-		)
-	)
 	(wire
 		(pts
@@
 		)
 	)
-	(wire
-		(pts
-			(xy 115.57 101.6) (xy 125.73 101.6)
-		)
-		(stroke
-			(width 0)
-			(type default)
-		)
-	)
 	(bus
 		(pts
@@
 	(wire
 		(pts
+			(xy 111.76 101.6) (xy 125.73 101.6)
+		)
+		(stroke
+			(width 0)
+			(type default)
+		)
+	)
+	(wire
+		(pts
 			(xy 151.13 124.46) (xy 151.13 127)
 		)
@@
 	(wire
 		(pts
-			(xy 148.59 124.46) (xy 148.59 134.62)
+			(xy 148.59 124.46) (xy 148.59 135.89)
 		)
 		(stroke
@@
 		)
 	)
-	(bus
-		(pts
-			(xy 182.88 96.52) (xy 182.88 137.16)
+	(wire
+		(pts
+			(xy 154.94 135.89) (xy 148.59 135.89)
 		)
 		(stroke
@@
 	(bus
 		(pts
-			(xy 151.13 137.16) (xy 148.59 137.16)
-		)
-		(stroke
-			(width 0)
-			(type default)
-		)
-	)
-	(bus
-		(pts
-			(xy 143.51 137.16) (xy 140.97 137.16)
+			(xy 140.97 143.51) (xy 140.97 140.97)
+		)
+		(stroke
+			(width 0)
+			(type default)
+		)
+	)
+	(bus
+		(pts
+			(xy 143.51 140.97) (xy 140.97 140.97)
 		)
 		(stroke
@@
 		)
 	)
-	(bus
-		(pts
-			(xy 146.05 137.16) (xy 143.51 137.16)
+	(wire
+		(pts
+			(xy 138.43 124.46) (xy 138.43 138.43)
+		)
+		(stroke
+			(width 0)
+			(type default)
+		)
+	)
+	(bus
+		(pts
+			(xy 146.05 140.97) (xy 143.51 140.97)
 		)
 		(stroke
@@
 		)
 	)
-	(label "ADC.CS"
-		(at 138.43 134.62 90)
+	(label "ADC_SPI.CS"
+		(at 138.43 138.43 90)
 		(effects
 			(font
@@
 		)
 	)
-	(label "ADC.MOSI"
-		(at 140.97 134.62 90)
+	(label "ADC_SPI.MOSI"
+		(at 140.97 138.43 90)
 		(effects
 			(font
@@
 		)
 	)
-	(label "ADC.MISO"
-		(at 146.05 134.62 90)
+	(label "ADC_SPI.MISO"
+		(at 146.05 138.43 90)
 		(effects
 			(font
@@
 		)
 	)
-	(label "ADC.CLK"
-		(at 143.51 134.62 90)
+	(label "ADC_SPI.CLK"
+		(at 143.51 138.43 90)
 		(effects
 			(font
@@
 		)
 	)
-	(hierarchical_label "ADC{RST DRDY MOSI MISO CLK CS START}"
+	(hierarchical_label "ADC.DRDY"
+		(shape input)
+		(at 154.94 135.89 0)
+		(effects
+			(font
+				(size 1.27 1.27)
+			)
+			(justify left)
+		)
+	)
+	(hierarchical_label "ADC.RST"
+		(shape input)
+		(at 185.42 99.06 0)
+		(effects
+			(font
+				(size 1.27 1.27)
+			)
+			(justify left)
+		)
+	)
+	(hierarchical_label "ADC.START"
+		(shape input)
+		(at 111.76 101.6 180)
+		(effects
+			(font
+				(size 1.27 1.27)
+			)
+			(justify right)
+		)
+	)
+	(hierarchical_label "ADC_SPI{MOSI MISO CLK CS}"
 		(shape bidirectional)
-		(at 182.88 96.52 0)
-		(effects
-			(font
-				(size 1.27 1.27)
-			)
-			(justify left)
+		(at 137.16 143.51 180)
+		(effects
+			(font
+				(size 1.27 1.27)
+			)
+			(justify right)
 		)
 	)
@@
 			)
 		)
-		(property "Footprint" ""
+		(property "Footprint" "Capacitor_SMD:C_0603_1608Metric_Pad1.08x0.95mm_HandSolder"
 			(at 128.27 56.1848 0)
 			(effects
@@
 			)
 		)
-		(property "Footprint" ""
+		(property "Footprint" "Capacitor_SMD:C_0603_1608Metric_Pad1.08x0.95mm_HandSolder"
 			(at 147.6248 53.34 0)
 			(effects
