File: hardware/UPP_simple/analog_inputs.kicad_sch (KiCad schematic)
At the start: 103 parts, among them J1 Conn_01x03, J10 Conn_01x03, J11 Conn_01x03, J12 Conn_01x03, J13 Conn_01x03, J14 Conn_01x03, J15 Conn_01x03, J16 Conn_01x03, J17 Conn_01x03, J18 Conn_01x03, J19 Conn_01x04, J2 Conn_01x03, J20 Conn_01x03, J21 Conn_01x03, J22 Conn_01x04, J23 Conn_01x03, J24 Conn_01x03, J25 Conn_01x04, J26 Conn_01x03, J27 Conn_01x03, J28 Conn_01x04, J29 Conn_01x04, J3 Conn_01x03, J30 Conn_01x04, J31 Conn_01x03, J32 Conn_01x03, J33 Conn_01x03, J34 Conn_01x03, J35 Conn_01x03, J36 Conn_01x03, J4 Conn_01x03, J5 Conn_01x03, J6 Conn_01x03, J7 Conn_01x03, J8 Conn_01x03, J9 Conn_01x03, U1 Opamp_Quad, U2 Opamp_Quad, U3 Opamp_Quad, U4 Opamp_Quad, U5 Opamp_Quad, U8 Opamp_Quad, U9 Opamp_Quad

Commit message: Add files via upload
Parts:
- removed J10, J11, J12, J13, J14, J15, J16, J17, J18, J20, J21, J23, J24, J26, J27, J31, J32, J33, J34, J35, J36, J7, J8, J9: Conn_01x03, symbol Connector_Generic:Conn_01x03
- removed J22, J25, J28, J29, J30: Conn_01x04, symbol Connector_Generic:Conn_01x04
- removed R16, R17, R20, R8: 0R, Resistor_SMD:R_0603_1608Metric, symbol Device:R_Small
- removed R16, R19, R20: 10k, Resistor_SMD:R_0603_1608Metric, symbol Device:R_Small
- removed R18, R19, R21 (x2): 14k, Resistor_SMD:R_0603_1608Metric, symbol Device:R_Small
- added J10, J11, J7, J8, J9: Conn_01x04, symbol Connector_Generic:Conn_01x04
- added JP1, JP10, JP11, JP12, JP13, JP14, JP15, JP16, JP17, JP18, JP19, JP2, JP20, JP21, JP22, JP23, JP24, JP3, JP4, JP5, JP6, JP7, JP8, JP9: Jumper_3_Open, symbol Jumper:Jumper_3_Open
- added R1, R20, R4, R7: 0R, Resistor_SMD:R_0603_1608Metric_Pad0.98x0.95mm_HandSolder, symbol Device:R_Small
- added R16, R2, R21, R5: 14k, Resistor_SMD:R_0603_1608Metric_Pad0.98x0.95mm_HandSolder, symbol Device:R_Small
- added R19, R3, R6: 10k, Resistor_SMD:R_0603_1608Metric_Pad0.98x0.95mm_HandSolder, symbol Device:R_Small
- R17, R18, R22, R23, R24, R25, R26, R27, R28, R29, R30, R32, R33, R36, R37, R41, R42, R43, R44, R45, R46, R8: footprint Resistor_SMD:R_0603_1608Metric -> Resistor_SMD:R_0603_1608Metric_Pad0.98x0.95mm_HandSolder
- R31, R38, R47, R48, R49: value 1k -> 3k92; footprint Resistor_SMD:R_0603_1608Metric -> Resistor_SMD:R_0603_1608Metric_Pad0.98x0.95mm_HandSolder
- R34, R39, R50, R52, R54: value 20k5 -> 1k; footprint Resistor_SMD:R_0603_1608Metric -> Resistor_SMD:R_0603_1608Metric_Pad0.98x0.95mm_HandSolder
- R35, R40, R51, R53, R55: value 3k92 -> 20k5; footprint Resistor_SMD:R_0603_1608Metric -> Resistor_SMD:R_0603_1608Metric_Pad0.98x0.95mm_HandSolder
Connections:
- net +12V: now also JP1.3 (B), JP11.3 (B), JP13.3 (B), JP15.3 (B), JP17.3 (B), JP19.3 (B), JP21.3 (B), JP23.3 (B), JP3.3 (B), JP5.3 (B), JP7.3 (B), JP9.3 (B); no longer J2.3 (Pin_3), J5.3 (Pin_3)
- net +5V: now also JP1.1 (A), JP11.1 (A), JP13.1 (A), JP15.1 (A), JP17.1 (A), JP19.1 (A), JP21.1 (A), JP23.1 (A), JP3.1 (A), JP5.1 (A), JP7.1 (A), JP9.1 (A); no longer J2.1 (Pin_1), J5.1 (Pin_1)
- net DIF2: now also R34.2; no longer R31.2
- net DIF3: now also R39.2; no longer R38.2
- net DIF4: now also R50.2; no longer R47.2
- net DIF5: now also R52.2; no longer R48.2
- net DIF6: now also R54.2; no longer R49.2
- net GND: now also J2.1 (Pin_1), J3.1 (Pin_1), J5.1 (Pin_1), J6.1 (Pin_1), R18.1, R22.1, R25.1, R29.1, R31.1, R38.1, R47.1, R48.1, R49.1, J10.1 (Pin_1), J11.1 (Pin_1), J7.1 (Pin_1), J8.1 (Pin_1), J9.1 (Pin_1), R19.1, R3.1, R6.1; no longer R18.2, R22.2, R25.2, R29.2, R34.2, R39.2, R50.2, R52.2, R54.2
- net at R36.2, U2.6 (-): now also R39.1; no longer R38.1
- net at R43.1: now also J10.3 (Pin_3)
- net at R43.2, U4.6 (-): now also R52.1; no longer R48.1
- net at R44.1: now also J10.2 (Pin_2)
- net at R44.2, U4.5 (+): now also JP22.2 (C)
- net at R37.2, U2.5 (+): now also JP18.2 (C)
- net at R30.1: now also JP14.1 (A)
- net at R28.2, U8.5 (+): now also JP14.2 (C)
- net at R33.2, U9.3 (+): now also R17.1, R18.2; no longer R17.2, R18.1
- net at U4.3 (+): now also R22.2, R20.2, R21.1; no longer R22.1
- net at R36.1: now also J8.3 (Pin_3)
- net at J19.4 (Pin_4): now also JP13.2 (C)
- net at R45.1: now also J11.3 (Pin_3)
- net at R45.2, U5.6 (-): now also R54.1; no longer R49.1
- net at R27.2, U1.5 (+): now also JP16.2 (C)
- net at R26.2, U1.6 (-): now also R34.1; no longer R31.1
- net at R46.1: now also J11.2 (Pin_2)
- net at R55.1: now also JP24.1 (A)
- net at J3.2 (Pin_2): now also JP8.2 (C)
- net at U1.3 (+): now also R1.2, R2.1, R3.2
- net at J3.3 (Pin_3): now also JP7.2 (C)
- net at U3.3 (+): now also R16.1, R19.2, R7.2
- net at J1.2 (Pin_2): now also JP4.2 (C); no longer J3.1 (Pin_1)
- net at J1.3 (Pin_3): now also JP3.2 (C); no longer J2.2 (Pin_2)
- net at R37.1: now also J8.2 (Pin_2)
- net at R27.1: now also J7.2 (Pin_2)
- net at R26.1: now also J7.3 (Pin_3)
- net at R23.2, U5.3 (+): now also R24.1, R25.2; no longer R24.2, R25.1
- net at J4.2 (Pin_2): now also JP2.2 (C); no longer J6.1 (Pin_1)
- net at J4.3 (Pin_3): now also JP1.2 (C); no longer J5.2 (Pin_2)
- net at R46.2, U5.5 (+): now also JP24.2 (C)
- net at R51.1: now also JP20.1 (A)
- net at R50.1: now also R41.2, U3.6 (-)
- net at R42.2, U3.5 (+): now also JP20.2 (C)
- net at R23.1: now also JP12.3 (B)
- net at R40.1: now also JP18.1 (A)
- net at U2.3 (+): now also R4.2, R5.1, R6.2
- net at R41.1: now also J9.3 (Pin_3)
- net at R33.1: now also JP2.3 (B); no longer J6.2 (Pin_2)
- net at R35.1: now also JP16.1 (A)
- net at J6.3 (Pin_3): now also JP11.2 (C); no longer R17.1
- net at R53.1: now also JP22.1 (A)
- net at R42.1: now also J9.2 (Pin_2)
- new net: J9.4 (Pin_4), JP19.2 (C)
- new net: JP4.3 (B), R1.1
- new net: J11.4 (Pin_4), JP23.2 (C)
- new net: J7.4 (Pin_4), JP15.2 (C)
- new net: JP14.3 (B), R29.2
- new net: JP2.1 (A), R17.2
- new net: JP10.1 (A), R21.2
- new net: J5.2 (Pin_2), JP10.2 (C)
- new net: JP10.3 (B), R20.1
- new net: JP8.1 (A), R16.2
- new net: J5.3 (Pin_3), JP9.2 (C)
- new net: JP8.3 (B), R7.1
- new net: JP24.3 (B), R49.2
- new net: JP4.1 (A), R2.2
- new net: J10.4 (Pin_4), JP21.2 (C)
- new net: J6.2 (Pin_2), JP12.2 (C)
- new net: JP6.3 (B), R4.1
- new net: J8.4 (Pin_4), JP17.2 (C)
- new net: JP18.3 (B), R38.2
- new net: J2.3 (Pin_3), JP5.2 (C)
- new net: JP20.3 (B), R47.2
- new net: JP16.3 (B), R31.2
- new net: JP6.1 (A), R5.2
- new net: JP12.1 (A), R24.2
- new net: JP22.3 (B), R48.2
- new net: J2.2 (Pin_2), JP6.2 (C)
